File: pcb/_autosave-keyboard.kicad_pcb (KiCad board)
At the start: 2 copper layers, 276.2 x 81 mm, 120 parts, among them J1 Conn_01x04_Pin, J2 AudioJack4, J3 USB_C_Receptacle_USB2.0_16P, J4 AudioJack4, J5 USB_C_Receptacle_USB2.0_16P, J6 Conn_01x04_Pin, SW1 SW_Push, SW10 SW_Push_45deg, SW11 SW_Push_45deg, SW12 SW_Push_45deg, SW13 SW_Push_45deg, SW14 SW_Push_45deg, SW15 SW_Push_45deg, SW16 SW_Push_45deg, SW17 SW_Push_45deg, SW18 SW_Push_45deg, SW19 SW_Push_45deg, SW2 SW_Push_45deg, SW20 SW_Push_45deg, SW21 SW_Push_45deg, SW22 SW_Push_45deg, SW26 SW_Push_45deg, SW27 SW_Push_45deg, SW28 SW_Push_45deg, SW29 SW_Push_45deg, SW3 SW_Push_45deg, SW30 SW_Push_45deg, SW31 SW_Push_45deg, SW32 SW_Push_45deg, SW33 SW_Push_45deg, SW34 SW_Push_45deg, SW35 SW_Push_45deg, SW39 SW_Push_45deg, SW4 SW_Push_45deg, SW40 SW_Push_45deg, SW41 SW_Push_45deg, SW42 SW_Push_45deg, SW43 SW_Push_45deg, SW44 SW_Push_45deg, SW45 SW_Push_45deg, SW46 SW_Push_45deg, SW48 SW_Push_45deg, SW49 SW_Push_45deg, SW5 SW_Push_45deg, SW50 SW_Push_45deg, SW51 SW_Push, SW6 SW_Push_45deg, SW7 SW_Push_45deg, SW8 SW_Push_45deg, SW9 SW_Push_45deg, U2 AMS1117-3.3, U4 STM32F072CBTx, U5 STM32F072CBTx, U6 AMS1117-3.3

Commit message: pogresss
Parts:
- moved J3 389.4 mm to (153.4, 42.5), turned to 180 degrees
- moved J5 364.6 mm to (184.3, 42.5), turned to 180 degrees
- moved J2 325.4 mm to (161.7, 53.3), turned to -90 degrees
- moved J4 323.1 mm to (176.0, 54.4), turned to 90 degrees
- moved U4 10.7 mm to (476.0, 171.1)
